File: Teensylu2-0.7.sch (EAGLE design)
At the start: 108 parts, among them IC2 AT90USB1286, J1 USB-MICRO-PTH, J2 39-29-3066, J3 MICROSD, P1 POLOLU-X, P2 POLOLU-Y, P3 POLOLU-Z, P4 POLOLU-E, P5 POLOLU-E, Q3 PMV45EN, Q5 PSMN1R2-30YLC, Q6 PSMN1R2-30YLC, Q7 PSMN1R2-30YLC, U1 LM2841, U2 PRTR5V0U4D, U7 AP7313, U8 TXB0104

Commit message: Alpha release
Caps have been moved over to SMD. Almost have all parts in the Teensylu
lib. Silkscreen is still incomplete. Switched to a new regulator. Added
attributes to all of the parts (haven't done all of the resistors yet,
but most others should have info like the manufacturer part #, etc.)
Parts:
- removed C32: 10uF, ipc-7351-capacitor:CAPACITOR_0805
- removed IC2: AT90USB1286, Atmel-at90usb-teensy:AT90USB
- removed JP25: FAN, SparkFun:M02POLAR
- removed JP26, JP33: FIDUCIAL1X2.5, SparkFun:FIDUCIAL1X2.5
- removed JP27: X-STOP, SparkFun:M03POLAR
- removed JP28: Y-STOP, SparkFun:M03POLAR
- removed JP29: Z-STOP, SparkFun:M03POLAR
- removed JP30: E-STOP, SparkFun:M03POLAR
- removed JP32: BOOT, teensylu:JUMPER-2PTH
- removed JP35: MOT-Z, SparkFun:M04POLAR
- removed JP40: (no value), teensylu:PROGHEADER
- removed Q5, Q6, Q7: PSMN1R2-30YLC, teensylu:PSMN1R2-30YLC
- removed R24: 10k, ipc-7351-resistor:RESISTOR_0603
- removed R25: 100, ipc-7351-resistor:RESISTOR_0603
- removed R26: 4.7k, ipc-7351-resistor:RESISTOR_0603
- removed R37: 5.6k, ipc-7351-resistor:RESISTOR_0603
- removed R38: 1k, ipc-7351-resistor:RESISTOR_0603
- removed U$51: 4P-TERM-BLOCK284391-4, teensylu:4P-TERM-BLOCK284391-4
- removed U7: AP7313, teensylu:AP7313
- removed U8: TXB0104, teensylu:TXB0104
- removed XTAL: KYOCERA_PQRC_TYPE_S_RESONATOR, Kyocera_Resonator:KYOCERA_PQRC_TYPE_S_RESONATOR
- added C12: 10pF, teensylu:CAPACITOR_0603
- added C19, C20, C21: 100uF, rcl:CPOL-USD
- added D2: SCH-DIODESOD123F, teensylu:SCH-DIODESOD123F
- added F1: MINISMDC050F1812, teensylu:MINISMDC050F1812
- added IC1: AT90USB1286, teensylu:AT90USB
- added J4: 39-29-3066, teensylu:39-29-3066
- added JP10: X-STOP, teensylu:M03POLAR
- added JP11: Y-STOP, teensylu:M03POLAR
- added JP12: E-STOP, teensylu:M03POLAR
- added JP15: (no value), teensylu:JUMPER-2PTH
- added JP16: MOT-X, teensylu:M04POLAR
- added JP17: MOT-Y, teensylu:M04POLAR
- added JP18, JP19: MOT-E, teensylu:M04POLAR
- added JP20: MOT-Z, teensylu:M04POLAR
- added JP9: Z-STOP, teensylu:M03POLAR
- added Q1: PMV45EN, teensylu:MOSFET-NCH_SOT-23
- added Q2, Q4: PSMN1R2-30YLCPOWERPACK-S08, teensylu:PSMN1R2-30YLCPOWERPACK-S08
- added R2: 10k, teensylu:RESISTOR_0603
- added R22: 100k, teensylu:RESISTOR_0603
- added R3: 100, teensylu:RESISTOR_0603
- added R4: 36k, teensylu:RESISTOR_0603
- added R5: 6.49, teensylu:RESISTOR_0603
- added U3: AP7313SOT23C, teensylu:AP7313SOT23C
- added U4: TXB0104TSSOP14, teensylu:TXB0104TSSOP14
- added X1: 16MHZ, teensylu:XTAL
- C1: value 100uf -> 4.7uF; device SparkFun:CAP_POLPTH1 -> teensylu:CAPACITOR_0805; VDC (none) -> 50v
- C10: device ipc-7351-capacitor:CAPACITOR_0603 -> teensylu:CAPACITOR_0805; ESR (none) -> 0.0030; VDC (none) -> 10v
- C11: value 1uf -> 10uF; device ipc-7351-capacitor:CAPACITOR_0603 -> teensylu:CAPACITOR_0603
- C13: value 0.1uF -> 10pF; device ipc-7351-capacitor:CAPACITOR_0603 -> teensylu:CAPACITOR_0603
- C14, C16: value 0.1uF -> 10uF; device ipc-7351-capacitor:CAPACITOR_0603 -> teensylu:CAPACITOR_0603
- C15: value 0.22uF -> 10uF; device ipc-7351-capacitor:CAPACITOR_0603 -> teensylu:CAPACITOR_0603
- C17: value 1uF -> 100uF; device ipc-7351-capacitor:CAPACITOR_0805 -> rcl:CPOL-USD; MANUFACTURER (none) -> Panasonic; MANUFACTURER_PART_NUMBER (none) -> EEE-FTH101XAP; TOLERANCE (none) -> 20%; VDC (none) -> 50v
- C18: MANUFACTURER (none) -> Panasonic; MANUFACTURER_PART_NUMBER (none) -> EEE-FTH101XAP; TOLERANCE (none) -> 20%; VDC (none) -> 50v
- C2: value 100uf -> 100uF; device SparkFun:CAP_POLPTH1 -> rcl:CPOL-USD; MANUFACTURER (none) -> Panasonic; MANUFACTURER_PART_NUMBER (none) -> EEE-FTH101XAP; TOLERANCE (none) -> 20%; VDC (none) -> 50v
- C3: value 100uf -> 0.1uF; device SparkFun:CAP_POLPTH1 -> teensylu:CAPACITOR_0603; VDC (none) -> 10v
- C4: value 100uf -> 100nF; device SparkFun:CAP_POLPTH1 -> teensylu:CAPACITOR_0603; ESR (none) -> 0.0064; VDC (none) -> 50
- C5: value 10uF -> 0.1uf; device ipc-7351-capacitor:CAPACITOR_0603 -> teensylu:CAPACITOR_0603
- C6: value 22uF -> 0.1uF; device ipc-7351-capacitor:CAPACITOR_0805 -> teensylu:CAPACITOR_0603; VDC (none) -> 10v
- C7: value 0.1uf -> 0.1uF; device ipc-7351-capacitor:CAPACITOR_0603 -> teensylu:CAPACITOR_0603; VDC (none) -> 10v
- C8: value 100uf -> 10uF; device SparkFun:CAP_POLPTH1 -> teensylu:CAPACITOR_0805; ESR (none) -> 0.0030; VDC (none) -> 10v
- C9: value 10uF -> 1uf; device ipc-7351-capacitor:CAPACITOR_0603 -> teensylu:CAPACITOR_0603
- D1: value SCH-DIODESMA -> SCH-DIODESOD123F; device printrbot:SCH-DIODESMA -> teensylu:SCH-DIODESOD123F; CURRENT (none) -> 1A; MANUFACTURER (none) -> NXP Semiconductors; MANUFACTURER_PART_NUMBER (none) -> PMEG4010CEH,115; REVERSE_VOLTAGE (none) -> 40V
- J1: value USB-MICRO-PTH -> MICROSD; device teensylu:USB-MICRO-PTH -> teensylu:MICROSD
- J2: value 39-29-3066 -> USB-MICRO-PTH; device teensylu:39-29-3066 -> teensylu:USB-MICRO-PTH
- J3: value MICROSD -> 4P-TERM-BLOCK284391-4; device teensylu:MICROSD -> teensylu:4P-TERM-BLOCK284391-4
- JP1: value MOT-X -> 12VPWR; device SparkFun:M04POLAR -> teensylu:M02POLAR
- JP2: value MOT-E -> FAN; device SparkFun:M04POLAR -> teensylu:M02POLAR
- JP3: value MOT-Y -> FIDUCIAL1X2.5; device SparkFun:M04POLAR -> SparkFun:FIDUCIAL1X2.5
- JP4: value JUMPER-3PTH -> FIDUCIAL1X2.5; device teensylu:JUMPER-3PTH -> SparkFun:FIDUCIAL1X2.5
- JP5: value JUMPER-3PTH -> BOOT; device teensylu:JUMPER-3PTH -> teensylu:JUMPER-2PTH
- JP6: value 12VPWR -> JUMPER-3PTH; device SparkFun:M02POLAR -> teensylu:JUMPER-3PTH
- JP7: value MOT-E -> (none); device SparkFun:M04POLAR -> teensylu:PROGHEADER
- JP8: value (none) -> JUMPER-3PTH; device teensylu:JUMPER-2PTH -> teensylu:JUMPER-3PTH
- L1: value 47uH -> 68uH; device teensylu:L-US -> teensylu:INDUCTORSRN6045; DCR (none) -> 0.351; IRMS (none) -> 0.9A; MANUFACTURER (none) -> Bourns; MANUFACTURER_PART_NUMBER (none) -> SRN6045-680M
- Q3: value PMV45EN -> PSMN1R2-30YLCPOWERPACK-S08; device ipc-7351-transistor:MOSFET-NCH_SOT-23 -> teensylu:PSMN1R2-30YLCPOWERPACK-S08
- R1, R12, R13, R14, R23, R7: device ipc-7351-resistor:RESISTOR_0603 -> teensylu:RESISTOR_0603
- R10: value 4.7k -> 10k; device ipc-7351-resistor:RESISTOR_0603 -> teensylu:RESISTOR_0603
- R11: value 10k -> 100; device ipc-7351-resistor:RESISTOR_0603 -> teensylu:RESISTOR_0603
- R15: value 100k -> 100; device ipc-7351-resistor:RESISTOR_0603 -> teensylu:RESISTOR_0603
- R16, R17, R18: value 100k -> 4.7k; device ipc-7351-resistor:RESISTOR_0603 -> teensylu:RESISTOR_0603
- R19, R20, R21: value 100 -> 100k; device ipc-7351-resistor:RESISTOR_0603 -> teensylu:RESISTOR_0603
- R6: value 10k -> 22; device ipc-7351-resistor:RESISTOR_0603 -> teensylu:RESISTOR_0603
- R8: value 22 -> 10k; device ipc-7351-resistor:RESISTOR_0603 -> teensylu:RESISTOR_0603
- R9: value 4.7k -> 100; device ipc-7351-resistor:RESISTOR_0603 -> teensylu:RESISTOR_0603
- U1: value LM2841 -> LMR16006X; device teensylu:LM2841 -> teensylu:LMR16006X
- U2: value PRTR5V0U4D -> PRTR5V0U4DSOT23-6; device teensylu:PRTR5V0U4D -> teensylu:PRTR5V0U4DSOT23-6
- renumbered JP21 to JP14, JP22 to JP13, JP31 to J6, U$15 to SJ12, U$17 to SCREW2, U$24 to SCREW3, U$27 to SJ7, U$33 to SJ2, U$34 to SCREW4, U$36 to J5, U$37 to SCREW1, U$43 to J8, U$50 to J7, U$53 to SJ13, U$54 to SJ8, U$55 to SJ3, U$56 to SJ14, U$57 to SJ9, U$58 to SJ4, U$59 to SJ15, U$60 to SJ10, U$61 to SJ5, U$62 to SJ16, U$63 to SJ11, U$64 to SJ6
Connections:
- new net N$5: F1.P$2, JP2.2
- net !E1-ENABLE: now also IC1.PC7_A15_IC3_CLK0, R22.2; no longer IC2.PC7_A15_IC3_CLK0, R17.2
- net !E2-ENABLE: now also IC1.PC1_A9; no longer IC2.PC1_A9
- net !HOTBED: now also IC1.PC4_A12_OC3C, R10.1; no longer IC2.PC4_A12_OC3C, R20.1
- net !HOTEND-1: now also IC1.PC5_A13_OC3B, R8.1, R9.1; no longer IC2.PC5_A13_OC3B, R19.1, R6.1
- net !HOTEND-2: now also IC1.PF3_ADC3, R14.1, R15.1; no longer IC2.PF3_ADC3, R24.1, R25.1
- net !PWM-FAN: now also IC1.PC6_A14_OC3A, R2.1, R3.1; no longer IC2.PC6_A14_OC3A, R14.1, R21.1
- net !RESET: now also IC1./RESET, JP7.2; no longer IC2./RESET, JP40.2
- net !X-ENABLE: now also IC1.PF7_ADC7_TDI, R20.2; no longer IC2.PF7_ADC7_TDI, R18.2
- net !Y-ENABLE: now also IC1.PA2_AD2, R19.2; no longer IC2.PA2_AD2, R15.2
- net !Z-ENABLE: now also IC1.PA5_AD5, R21.2; no longer IC2.PA5_AD5, R16.2
- net +3V3: now also C11.1, J1.VDD, U3.OUT, U4.OE, U4.VCCA; no longer C32.1, J3.VDD, U7.OUT, U8.OE, U8.VCCA
- net 12V: now also C1.1, C17.+, C19.+, C20.+, C21.+, J3.1, J3.2, J4-1_+V.S, J4-2_+V.S, J4-3_+V.S, JP1.1, JP2.1, JP8.1; no longer C1.+, C17.1, C3.+, C4.+, C8.+, J2-1_+V.S, J2-2_+V.S, J2-3_+V.S, JP25.1, JP4.1, JP5.1, U$51.1, U$51.2
- net 5V: now also C10.1, C3.1, C6.2, C7.2, C8.1, IC1.AREF, IC1.AVCC, IC1.VCC, IC1.VCC@1, JP6.3, JP7.5, JP8.3, R16.2, R17.2, R18.2, R19.1, R20.1, R21.1, R22.1, R4.1, U3.IN, U4.VCCB; no longer C13.2, C14.1, C16.2, C6.1, IC2.AREF, IC2.AVCC, IC2.VCC, IC2.VCC@1, JP4.3, JP40.5, JP5.3, R10.2, R15.1, R16.1, R17.1, R18.1, R26.2, R37.1, R9.2, U7.IN, U8.VCCB
- net 5VREG_CB: now also C4.2; no longer C15.2
- net 5VREG_FB: now also R4.2, R5.1; no longer R37.2, R38.1
- net 5VREG_SW: now also C4.1; no longer C15.1
- net A4: now also IC1.PF4_ADC4_TCK; no longer IC2.PF4_ADC4_TCK
- net A5: now also IC1.PF5_ADC5_TMS; no longer IC2.PF5_ADC5_TMS
- net A6: now also IC1.PF6_ADC6_TDO; no longer IC2.PF6_ADC6_TDO
- net ALE: now also IC1.PE2_ALE_HWB, JP5.1; no longer IC2.PE2_ALE_HWB, JP32.1
- net B-THERM: now also C15.2, IC1.PF0_ADC0, R17.1; no longer C9.2, IC2.PF0_ADC0, R10.1
- net E-MOT-1A: now also JP18.2; no longer JP7.3
- net E-MOT-1A1: now also JP19.2; no longer JP2.3
- net E-MOT-1B: now also JP18.1; no longer JP7.4
- net E-MOT-1B1: now also JP19.1; no longer JP2.4
- net E-MOT-2A: now also JP18.3; no longer JP7.2
- net E-MOT-2A1: now also JP19.3; no longer JP2.2
- net E-MOT-2B: now also JP18.4; no longer JP7.1
- net E-MOT-2B1: now also JP19.4; no longer JP2.1
- net E-STOP: now also IC1.PE4_INT4_TOSC1, JP12.1; no longer IC2.PE4_INT4_TOSC1, JP30.1
- net E1-DIR: now also IC1.PC3_A11_T3; no longer IC2.PC3_A11_T3
- net E1-STEP: now also IC1.PC2_A10; no longer IC2.PC2_A10
- net E1-THERM: now also C14.2, IC1.PF1_ADC1, R16.1; no longer C10.2, IC2.PF1_ADC1, R9.1
- net E2-DIR: now also IC1.PC0_A8; no longer IC2.PC0_A8
- net E2-STEP: now also IC1.PE1_/RD; no longer IC2.PE1_/RD
- net E2-THERM: now also C16.2, IC1.PF2_ADC2, JP15.1, R18.1; no longer C5.2, IC2.PF2_ADC2, JP8.1, R26.1
- net ENDSTOP+V: now also JP10.2, JP11.2, JP12.2, JP6.2; no longer JP27.2, JP28.2, JP30.2, JP5.2
- net GND: now also C1.2, C10.2, C11.2, C12.1, C14.1, C15.1, C17.-, C19.-, C20.-, C21.-, C3.2, C6.1, C8.2, D2.A, IC1.AGND, IC1.GND, IC1.GND@1, IC1.UGND, J1.CD1, J1.SHEILD@1, J1.SHIELD@2, J1.SHIELD@3, J1.SHIELD@4, J2.GND, J3.3, J3.4, J4-4_GND.S, J4-5_GND.S, J4-6_GND.S, JP1.2, JP10.3, JP11.3, JP12.3, JP15.2, JP5.2, JP7.1, JP9.3, Q1.S, Q2.S1, Q2.S2, Q2.S3, Q3.S1, Q3.S2, Q3.S3, Q4.S1, Q4.S2, Q4.S3, R10.2, R2.2, R5.2, R8.2, U3.GND, U4.GND; no longer C1.-, C10.1, C11.1, C14.2, C17.2, C3.-, C32.2, C4.-, C6.2, C8.-, IC2.AGND, IC2.GND, IC2.GND@1, IC2.UGND, J2-4_GND.S, J2-5_GND.S, J2-6_GND.S, J3.CD1, J3.GND, J3.SHEILD@1, J3.SHIELD@2, J3.SHIELD@3, J3.SHIELD@4, JP27.3, JP28.3, JP29.3, JP30.3, JP32.2, JP40.1, JP6.2, JP8.2, Q3.S, Q5.S1, Q5.S2, Q5.S3, Q6.S1, Q6.S2, Q6.S3, Q7.S1, Q7.S2, Q7.S3, R11.2, R24.2, R38.2, R6.2, U$51.3, U$51.4, U7.GND, U8.GND, XTAL.GND
- net HOTBED-GND: now also Q3.D; no longer Q6.D
- net HOTEND-GND: now also Q2.D; no longer Q5.D
- net HOTEND-GND1: now also Q4.D; no longer Q7.D
- net MISO: now also IC1.PB3_PDO_PCINT3_MISO, JP7.6, U4.B1; no longer IC2.PB3_PDO_PCINT3_MISO, JP40.6, U8.B1
- net MOSI: now also IC1.PB2_PDI_PCINT2_MOSI, JP7.3, U4.B3; no longer IC2.PB2_PDI_PCINT2_MOSI, JP40.3, U8.B3
- net N$10: now also Q1.G, R3.2; no longer Q3.G, R21.2
- net N$11: now also Q2.G, R9.2; no longer Q5.G, R19.2
- net N$13: now also Q4.G, R15.2; no longer Q7.G, R25.2
- net N$2: now also Q3.G, R11.2; no longer Q6.G, R20.2
- net N$3: now also IC1.D-, R6.2; no longer IC2.D-, R7.2
- net N$4: now also IC1.D+, R7.2; no longer IC2.D+, R8.2
- net N$6: now also D2.C, F1.P$1, Q1.D; no longer JP25.2, Q3.D
- net PB4: now also IC1.PB4_PCINT4_OC2A; no longer IC2.PB4_PCINT4_OC2A
- net PD0-SCL: now also IC1.PD0_OC0B_SCL_INT0; no longer IC2.PD0_OC0B_SCL_INT0
- net PD1-SDA: now also IC1.PD1_OC2B_SDA_INT1; no longer IC2.PD1_OC2B_SDA_INT1
- net PD2-RX1: now also IC1.PD2_RXD1_INT2; no longer IC2.PD2_RXD1_INT2
- net PD3-TX1: now also IC1.PD3_TXD1_INT3; no longer IC2.PD3_TXD1_INT3
- net PD4: now also IC1.PD4_ICP1; no longer IC2.PD4_ICP1
- net PD5: now also IC1.PD5_XCK1; no longer IC2.PD5_XCK1
- net PD6: now also IC1.PD6_T1; no longer IC2.PD6_T1
- net PD7: now also IC1.PD7_T0; no longer IC2.PD7_T0
- net PE0: now also IC1.PE0_/WR; no longer IC2.PE0_/WR
- net PE5: now also IC1.PE5_INT5_TOSC2; no longer IC2.PE5_INT5_TOSC2
- net PE6: now also IC1.PE6_INT6_AIN0; no longer IC2.PE6_INT6_AIN0
- net PE7: now also IC1.PE7_INT7_AIN1_UVCON; no longer IC2.PE7_INT7_AIN1_UVCON
- net SCLK: now also IC1.PB1_PCINT1_SCLK, JP7.4, U4.B2; no longer IC2.PB1_PCINT1_SCLK, JP40.4, U8.B2
- net SDCD: now also IC1.PB7_PCINT7_OC0A_OC1C, J1.CD2; no longer IC2.PB7_PCINT7_OC0A_OC1C, J3.CD2
- net SDCLK: now also J1.CLK, U4.A2; no longer J3.CLK, U8.A2
- net SDCS: now also IC1.PB0_SS_PCINT0, U4.B4; no longer IC2.PB0_SS_PCINT0, U8.B4
- net SDCSH: now also J1.DAT3/CS, U4.A4; no longer J3.DAT3/CS, U8.A4
- net SDDI: now also J1.CMD/DI, U4.A3; no longer J3.CMD/DI, U8.A3
- net SDDO: now also J1.DAT0/DO, U4.A1; no longer J3.DAT0/DO, U8.A1
- net UCAP: now also C9.2, IC1.UCAP; no longer C11.2, IC2.UCAP
- net USB_DN: now also J2.D-, R6.1; no longer J1.D-, R7.1
- net USB_DP: now also J2.D+, R7.1; no longer J1.D+, R8.1
- net VBUS: now also C5.2, IC1.UVCC, IC1.VBUS, J2.VBUS; no longer C7.2, IC2.UVCC, IC2.VBUS, J1.VBUS
- net X-DIR: now also IC1.PA0_AD0; no longer IC2.PA0_AD0
- net X-MOT-1A: now also JP16.2; no longer JP1.3
- net X-MOT-1B: now also JP16.1; no longer JP1.4
- net X-MOT-2A: now also JP16.3; no longer JP1.2
- net X-MOT-2B: now also JP16.4; no longer JP1.1
- net X-STEP: now also IC1.PA1_AD1; no longer IC2.PA1_AD1
- net X-STOP: now also IC1.PB6_PCINT6_OC1B, JP10.1; no longer IC2.PB6_PCINT6_OC1B, JP27.1
- net XTAL1: now also C13.2, IC1.XTAL1, X1.2; no longer IC2.XTAL1, XTAL.1
- net XTAL2: now also C12.2, IC1.XTAL2, X1.1; no longer IC2.XTAL2, XTAL.2
- net Y-DIR: now also IC1.PA3_AD3; no longer IC2.PA3_AD3
- net Y-MOT-1A: now also JP17.2; no longer JP3.3
- net Y-MOT-1B: now also JP17.1; no longer JP3.4
- net Y-MOT-2A: now also JP17.3; no longer JP3.2
- net Y-MOT-2B: now also JP17.4; no longer JP3.1
- net Y-STEP: now also IC1.PA4_AD4; no longer IC2.PA4_AD4
- net Y-STOP: now also IC1.PB5_PCINT5_OC1A, JP11.1; no longer IC2.PB5_PCINT5_OC1A, JP28.1
- net Z-DIR: now also IC1.PA6_AD6; no longer IC2.PA6_AD6
- net Z-MOT-1A: now also JP20.2; no longer JP35.3
- net Z-MOT-1B: now also JP20.1; no longer JP35.4
- net Z-MOT-2A: now also JP20.3; no longer JP35.2
- net Z-MOT-2B: now also JP20.4; no longer JP35.1
- net Z-STEP: now also IC1.PA7_AD7; no longer IC2.PA7_AD7
- net Z-STOP: now also IC1.PE3_IUID, JP9.1; no longer IC2.PE3_IUID, JP29.1
- net Z-STOP-SUPPLY: now also JP8.2, JP9.2; no longer JP29.2, JP4.2
Other:
- moved on the sheet: C10, C11, C13, C14, C15, C16, C18, C2, C5, C6, C7, C9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
